Commit message: some extra stuff for indoor i fogor

File: src/vehicle_simulator/urdf/robot.urdf (copy).xacro (robot description, xacro)
@@ -18,14 +18,8 @@
     </visual>
     <inertial>
-      <mass value="100" />
+      <mass value="1e-5" />
       <origin xyz="0 0 0" rpy="0 0 0"/>
-      <inertia ixx="100" ixy="0" ixz="0" iyy="100" iyz="0" izz="100" />
+      <inertia ixx="1e-6" ixy="0" ixz="0" iyy="1e-6" iyz="0" izz="1e-6" />
     </inertial>
-    <collision>
-      <origin xyz="0 0 0" />
-      <geometry>
-        <box size="0.6 0.4 0.3"/>
-      </geometry>
-    </collision>
   </link>
   <joint name="base_link_joint" type="fixed">
